File: PCB/WhoopDock.kicad_pcb (KiCad board)
At the start: 2 copper layers, 35 parts, among them J1 BetaFPV_BT2.0, SW1 SW_Push, U1 ESP32-S3-WROOM-1, U2 CH224K, U3 XL1509-5.0E1, U4 BQ25890RTWR, U5 RT9193-33GB

Commit message: PCB Done
Parts:
- removed SW1: SW_Push, Button_Switch_THT:SW_PUSH_6mm_H5mm
- added BUZZER1: MLT-8530, easyeda2kicad:BUZ-SMD_4P-L8.5-W8.5-P8.50-BR, B.Cu at (178.2, 131.5)
- added C12: 10uF, Capacitor_SMD:C_0805_2012Metric, F.Cu at (202.0, 110.5)
- added C13: 47nF, Capacitor_SMD:C_0603_1608Metric, F.Cu at (213.8, 107.5)
- added C14: 10uF, Capacitor_SMD:C_0805_2012Metric, F.Cu at (201.8, 100.7)
- added C15: 10uF, Capacitor_SMD:C_0805_2012Metric, F.Cu at (201.9, 104.1)
- added C16: 10uF, Capacitor_SMD:C_0805_2012Metric, F.Cu at (215.1, 103.4)
- added C17: 4.7uF, Capacitor_SMD:C_0603_1608Metric, F.Cu at (214.6, 105.2)
- added C18: 1uF, Capacitor_SMD:C_0603_1608Metric, F.Cu at (216.0, 100.9)
- added C19: 10uF, Capacitor_SMD:C_0805_2012Metric, F.Cu at (221.6, 110.5)
- added C20: 1uF, Capacitor_SMD:C_0603_1608Metric, F.Cu at (235.7, 100.9)
- added C21: 47nF, Capacitor_SMD:C_0603_1608Metric, F.Cu at (233.5, 107.5)
- added C22: 4.7uF, Capacitor_SMD:C_0603_1608Metric, F.Cu at (234.2, 105.2)
- added C23: 10uF, Capacitor_SMD:C_0805_2012Metric, F.Cu at (234.8, 103.4)
- added C24: 10uF, Capacitor_SMD:C_0805_2012Metric, F.Cu at (221.5, 100.7)
- added C25: 10uF, Capacitor_SMD:C_0805_2012Metric, F.Cu at (221.5, 104.1)
- added C26: 10uF, Capacitor_SMD:C_0805_2012Metric, F.Cu at (241.2, 110.5)
- added C27: 1uF, Capacitor_SMD:C_0603_1608Metric, F.Cu at (255.3, 100.9)
- added C28: 47nF, Capacitor_SMD:C_0603_1608Metric, F.Cu at (253.1, 107.5)
- added C29: 4.7uF, Capacitor_SMD:C_0603_1608Metric, F.Cu at (253.8, 105.2)
- added C30: 10uF, Capacitor_SMD:C_0805_2012Metric, F.Cu at (254.4, 103.4)
- added C31: 10uF, Capacitor_SMD:C_0805_2012Metric, F.Cu at (241.1, 100.7)
- added C32: 10uF, Capacitor_SMD:C_0805_2012Metric, F.Cu at (241.1, 104.1)
- added C33: 10uF, Capacitor_SMD:C_0805_2012Metric, F.Cu at (209.4, 133.5)
- added C34: 1uF, Capacitor_SMD:C_0603_1608Metric, F.Cu at (195.3, 143.1)
- added C35: 47nF, Capacitor_SMD:C_0603_1608Metric, F.Cu at (197.5, 136.6)
- added C36: 4.7uF, Capacitor_SMD:C_0603_1608Metric, F.Cu at (196.8, 138.8)
- added C37: 10uF, Capacitor_SMD:C_0805_2012Metric, F.Cu at (196.3, 140.6)
- added C38: 10uF, Capacitor_SMD:C_0805_2012Metric, F.Cu at (209.5, 143.3)
- added C39: 10uF, Capacitor_SMD:C_0805_2012Metric, F.Cu at (209.5, 139.9)
- added C40: 10uF, Capacitor_SMD:C_0805_2012Metric, F.Cu at (229.0, 133.5)
- added C41: 1uF, Capacitor_SMD:C_0603_1608Metric, F.Cu at (215.0, 143.1)
- added C42: 47nF, Capacitor_SMD:C_0603_1608Metric, F.Cu at (217.2, 136.6)
- added C43: 4.7uF, Capacitor_SMD:C_0603_1608Metric, F.Cu at (216.4, 138.8)
- added C44: 10uF, Capacitor_SMD:C_0805_2012Metric, F.Cu at (215.9, 140.6)
- added C45: 10uF, Capacitor_SMD:C_0805_2012Metric, F.Cu at (229.2, 143.3)
- added C46: 10uF, Capacitor_SMD:C_0805_2012Metric, F.Cu at (229.2, 139.9)
- added C47: 10uF, Capacitor_SMD:C_0805_2012Metric, F.Cu at (248.7, 133.5)
- added C48: 1uF, Capacitor_SMD:C_0603_1608Metric, F.Cu at (234.6, 143.1)
- added C49: 47nF, Capacitor_SMD:C_0603_1608Metric, F.Cu at (236.8, 136.6)
- added C50: 4.7uF, Capacitor_SMD:C_0603_1608Metric, F.Cu at (236.1, 138.8)
- added C51: 10uF, Capacitor_SMD:C_0805_2012Metric, F.Cu at (235.5, 140.6)
- added C52: 10uF, Capacitor_SMD:C_0805_2012Metric, F.Cu at (248.8, 143.3)
- added C53: 10uF, Capacitor_SMD:C_0805_2012Metric, F.Cu at (248.8, 139.9)
- added C54: 10uF, Capacitor_SMD:C_0805_2012Metric, F.Cu at (184.4, 123.5)
- added C55: 0.1uF, Capacitor_SMD:C_0603_1608Metric, F.Cu at (184.2, 121.7)
- added C56: 10uF, Capacitor_SMD:C_0805_2012Metric, F.Cu at (160.9, 98.3)
- added C57: 10nF, Capacitor_SMD:C_0603_1608Metric, F.Cu at (164.2, 100.5)
- added C58: 10uF, Capacitor_SMD:C_0805_2012Metric, F.Cu at (166.7, 98.2)
- added D2: 1N4148W, Diode_SMD:D_SOD-123F, F.Cu at (178.2, 135.5)
- added J2: BetaFPV_BT2.0, easyeda2kicad:BetaFPV BT2.0, F.Cu at (225.3, 109.6)
- added J3: BetaFPV_BT2.0, easyeda2kicad:BetaFPV BT2.0, F.Cu at (244.9, 109.6)
- added J4: BetaFPV_BT2.0, easyeda2kicad:BetaFPV BT2.0, F.Cu at (205.7, 134.4)
- added J5: BetaFPV_BT2.0, easyeda2kicad:BetaFPV BT2.0, F.Cu at (225.3, 134.4)
- added J6: BetaFPV_BT2.0, easyeda2kicad:BetaFPV BT2.0, F.Cu at (244.9, 134.4)
- added L2: 1.5uH, Inductor_SMD:L_APV_APH0420, F.Cu at (210.7, 107.6)
- added L3: 1.5uH, Inductor_SMD:L_APV_APH0420, F.Cu at (230.3, 107.6)
- added L4: 1.5uH, Inductor_SMD:L_APV_APH0420, F.Cu at (250.0, 107.6)
- added L5: 1.5uH, Inductor_SMD:L_APV_APH0420, F.Cu at (200.7, 136.4)
- added L6: 1.5uH, Inductor_SMD:L_APV_APH0420, F.Cu at (220.3, 136.4)
- added L7: 1.5uH, Inductor_SMD:L_APV_APH0420, F.Cu at (239.9, 136.4)
- added M1: Fan, easyeda2kicad:Fan, F.Cu at (160.1, 105.0)
- added Q1: AO3400A, Package_TO_SOT_SMD:SOT-23, F.Cu at (217.0, 115.4)
- added Q10: AO4407A, easyeda2kicad:SOIC-8_L4.9-W3.9-P1.27-LS6.0-BL, F.Cu at (205.8, 141.5)
- added Q11: AO3400A, Package_TO_SOT_SMD:SOT-23, F.Cu at (214.0, 128.6)
- added Q12: AO4407A, easyeda2kicad:SOIC-8_L4.9-W3.9-P1.27-LS6.0-BL, F.Cu at (225.5, 141.5)
- added Q13: AO3400A, Package_TO_SOT_SMD:SOT-23, F.Cu at (233.6, 128.6)
- added Q14: AO4407A, easyeda2kicad:SOIC-8_L4.9-W3.9-P1.27-LS6.0-BL, F.Cu at (245.1, 141.5)
- added Q2: AO4407A, easyeda2kicad:SOIC-8_L4.9-W3.9-P1.27-LS6.0-BL, F.Cu at (205.5, 102.5)
- added Q3: AO3400A, Package_TO_SOT_SMD:SOT-23, F.Cu at (177.9, 132.5)
- added Q4: AO3400A, Package_TO_SOT_SMD:SOT-23, F.Cu at (163.0, 105.1)
- added Q5: AO3400A, Package_TO_SOT_SMD:SOT-23, F.Cu at (236.7, 115.4)
- added Q6: AO4407A, easyeda2kicad:SOIC-8_L4.9-W3.9-P1.27-LS6.0-BL, F.Cu at (225.2, 102.5)
- added Q7: AO3400A, Package_TO_SOT_SMD:SOT-23, F.Cu at (256.3, 115.4)
- added Q8: AO4407A, easyeda2kicad:SOIC-8_L4.9-W3.9-P1.27-LS6.0-BL, F.Cu at (244.8, 102.5)
- added Q9: AO3400A, Package_TO_SOT_SMD:SOT-23, F.Cu at (194.3, 128.6)
- added R14: 100, Resistor_SMD:R_0603_1608Metric, F.Cu at (211.8, 97.8)
- added R15: 5.1k, Resistor_SMD:R_0603_1608Metric, F.Cu at (214.8, 97.8)
- added R16: 5.1k, Resistor_SMD:R_0603_1608Metric, F.Cu at (216.3, 111.2)
- added R17: 5.1k, Resistor_SMD:R_0603_1608Metric, F.Cu at (215.3, 109.7)
- added R18: 10k, Resistor_SMD:R_0603_1608Metric, F.Cu at (215.4, 107.5)
- added R19: 10k, Resistor_SMD:R_0603_1608Metric, F.Cu at (208.7, 97.7)
- added R20: 15, Resistor_SMD:R_2512_6332Metric, F.Cu at (211.5, 118.7)
- added R21: 15, Resistor_SMD:R_2512_6332Metric, F.Cu at (211.5, 114.8)
- added R22: 15, Resistor_SMD:R_2512_6332Metric, F.Cu at (203.8, 118.7)
- added R23: 15, Resistor_SMD:R_2512_6332Metric, F.Cu at (203.8, 114.8)
- added R24: 5.1k, Resistor_SMD:R_0603_1608Metric, F.Cu at (217.0, 119.5)
- added R25: 100, Resistor_SMD:R_0603_1608Metric, F.Cu at (217.0, 121.1)
- added R26: 100, Resistor_SMD:R_0603_1608Metric, F.Cu at (175.2, 132.5)
- added R27: 100, Resistor_SMD:R_0603_1608Metric, F.Cu at (163.0, 107.9)
- added R28: 100, Resistor_SMD:R_0603_1608Metric, F.Cu at (236.7, 121.1)
- added R29: 100, Resistor_SMD:R_0603_1608Metric, F.Cu at (231.4, 97.8)
- added R30: 5.1k, Resistor_SMD:R_0603_1608Metric, F.Cu at (236.7, 119.5)
- added R31: 10k, Resistor_SMD:R_0603_1608Metric, F.Cu at (228.4, 97.7)
- added R32: 5.1k, Resistor_SMD:R_0603_1608Metric, F.Cu at (234.4, 97.8)
- added R33: 10k, Resistor_SMD:R_0603_1608Metric, F.Cu at (235.0, 107.5)
- added R34: 15, Resistor_SMD:R_2512_6332Metric, F.Cu at (223.4, 114.8)
- added R35: 15, Resistor_SMD:R_2512_6332Metric, F.Cu at (223.4, 118.7)
- added R36: 15, Resistor_SMD:R_2512_6332Metric, F.Cu at (231.2, 114.8)
- added R37: 15, Resistor_SMD:R_2512_6332Metric, F.Cu at (231.2, 118.7)
- added R38: 5.1k, Resistor_SMD:R_0603_1608Metric, F.Cu at (235.9, 111.2)
- added R39: 5.1k, Resistor_SMD:R_0603_1608Metric, F.Cu at (235.0, 109.7)
- added R40: 100, Resistor_SMD:R_0603_1608Metric, F.Cu at (256.3, 121.1)
- added R41: 100, Resistor_SMD:R_0603_1608Metric, F.Cu at (251.0, 97.8)
- added R42: 5.1k, Resistor_SMD:R_0603_1608Metric, F.Cu at (256.3, 119.5)
- added R43: 10k, Resistor_SMD:R_0603_1608Metric, F.Cu at (248.0, 97.7)
- added R44: 5.1k, Resistor_SMD:R_0603_1608Metric, F.Cu at (254.1, 97.8)
- added R45: 10k, Resistor_SMD:R_0603_1608Metric, F.Cu at (254.6, 107.5)
- added R46: 15, Resistor_SMD:R_2512_6332Metric, F.Cu at (243.1, 114.8)
- added R47: 15, Resistor_SMD:R_2512_6332Metric, F.Cu at (243.1, 118.7)
- added R48: 15, Resistor_SMD:R_2512_6332Metric, F.Cu at (250.8, 114.8)
- added R49: 15, Resistor_SMD:R_2512_6332Metric, F.Cu at (250.8, 118.7)
- added R50: 5.1k, Resistor_SMD:R_0603_1608Metric, F.Cu at (255.6, 111.2)
- added R51: 5.1k, Resistor_SMD:R_0603_1608Metric, F.Cu at (254.6, 109.7)
- added R52: 100, Resistor_SMD:R_0603_1608Metric, F.Cu at (194.3, 122.9)
- added R53: 100, Resistor_SMD:R_0603_1608Metric, F.Cu at (199.6, 146.2)
- added R54: 5.1k, Resistor_SMD:R_0603_1608Metric, F.Cu at (194.3, 124.5)
- added R55: 10k, Resistor_SMD:R_0603_1608Metric, F.Cu at (202.7, 146.3)
- added R56: 5.1k, Resistor_SMD:R_0603_1608Metric, F.Cu at (196.6, 146.2)
- added R57: 10k, Resistor_SMD:R_0603_1608Metric, F.Cu at (196.0, 136.5)
- added R58: 15, Resistor_SMD:R_2512_6332Metric, F.Cu at (207.6, 129.2)
- added R59: 15, Resistor_SMD:R_2512_6332Metric, F.Cu at (207.6, 125.3)
- added R60: 15, Resistor_SMD:R_2512_6332Metric, F.Cu at (199.9, 129.2)
- added R61: 15, Resistor_SMD:R_2512_6332Metric, F.Cu at (199.9, 125.3)
- added R62: 5.1k, Resistor_SMD:R_0603_1608Metric, F.Cu at (195.1, 132.8)
- added R63: 5.1k, Resistor_SMD:R_0603_1608Metric, F.Cu at (196.0, 134.3)
- added R64: 100, Resistor_SMD:R_0603_1608Metric, F.Cu at (214.0, 122.9)
- added R65: 100, Resistor_SMD:R_0603_1608Metric, F.Cu at (219.2, 146.2)
- added R66: 5.1k, Resistor_SMD:R_0603_1608Metric, F.Cu at (214.0, 124.5)
- added R67: 10k, Resistor_SMD:R_0603_1608Metric, F.Cu at (222.3, 146.3)
- added R68: 5.1k, Resistor_SMD:R_0603_1608Metric, F.Cu at (216.2, 146.2)
- added R69: 10k, Resistor_SMD:R_0603_1608Metric, F.Cu at (215.7, 136.5)
- added R70: 15, Resistor_SMD:R_2512_6332Metric, F.Cu at (227.2, 129.2)
- added R71: 15, Resistor_SMD:R_2512_6332Metric, F.Cu at (227.2, 125.3)
- added R72: 15, Resistor_SMD:R_2512_6332Metric, F.Cu at (219.5, 129.2)
- added R73: 15, Resistor_SMD:R_2512_6332Metric, F.Cu at (219.5, 125.3)
- added R74: 5.1k, Resistor_SMD:R_0603_1608Metric, F.Cu at (214.7, 132.8)
- added R75: 5.1k, Resistor_SMD:R_0603_1608Metric, F.Cu at (215.7, 134.3)
- added R76: 100, Resistor_SMD:R_0603_1608Metric, F.Cu at (233.6, 122.9)
- added R77: 100, Resistor_SMD:R_0603_1608Metric, F.Cu at (238.9, 146.2)
- added R78: 5.1k, Resistor_SMD:R_0603_1608Metric, F.Cu at (233.6, 124.5)
- added R79: 10k, Resistor_SMD:R_0603_1608Metric, F.Cu at (241.9, 146.3)
- added R80: 5.1k, Resistor_SMD:R_0603_1608Metric, F.Cu at (235.8, 146.2)
- added R81: 10k, Resistor_SMD:R_0603_1608Metric, F.Cu at (235.3, 136.5)
- added R82: 15, Resistor_SMD:R_2512_6332Metric, F.Cu at (246.8, 129.2)
- added R83: 15, Resistor_SMD:R_2512_6332Metric, F.Cu at (246.8, 125.3)
- added R84: 15, Resistor_SMD:R_2512_6332Metric, F.Cu at (239.1, 129.2)
- added R85: 15, Resistor_SMD:R_2512_6332Metric, F.Cu at (239.1, 125.3)
- added R86: 5.1k, Resistor_SMD:R_0603_1608Metric, F.Cu at (234.3, 132.8)
- added R87: 5.1k, Resistor_SMD:R_0603_1608Metric, F.Cu at (235.3, 134.3)
- added R88: 5.1k, Resistor_SMD:R_0603_1608Metric, F.Cu at (193.1, 110.2)
- added R89: 5.1k, Resistor_SMD:R_0603_1608Metric, F.Cu at (191.5, 110.2)
- added R90: 5.1k, Resistor_SMD:R_0603_1608Metric, F.Cu at (191.6, 121.1)
- added R91: 0, Resistor_SMD:R_0603_1608Metric, F.Cu at (164.2, 102.0)
- added SW2: SW_Push, Button_Switch_THT:SW_PUSH_6mm_H5mm, F.Cu at (168.0, 138.5)
- added SW3: SW_Push, Button_Switch_THT:SW_PUSH_6mm_H5mm, F.Cu at (180.4, 138.5)
- added U10: BQ25890_1, easyeda2kicad:WQFN-24_L4.0-W4.0-P0.50-BL-EP, F.Cu at (200.2, 143.2)
- added U11: BQ25890_1, easyeda2kicad:WQFN-24_L4.0-W4.0-P0.50-BL-EP, F.Cu at (219.8, 143.2)
- added U12: BQ25890_1, easyeda2kicad:WQFN-24_L4.0-W4.0-P0.50-BL-EP, F.Cu at (239.4, 143.2)
- added U13: RT9193-33GB, easyeda2kicad:SOT-23-5_L3.0-W1.7-P0.95-LS2.8-BL, F.Cu at (163.7, 98.2)
- added U6: ~, easyeda2kicad:1.3 TFT, F.Cu at (177.5, 100.0)
- added U7: TCA9548APWR, Package_SO:TSSOP-24_4.4x7.8mm_P0.65mm, F.Cu at (194.5, 116.4)
- added U8: BQ25890_1, easyeda2kicad:WQFN-24_L4.0-W4.0-P0.50-BL-EP, F.Cu at (230.8, 100.8)
- added U9: BQ25890_1, easyeda2kicad:WQFN-24_L4.0-W4.0-P0.50-BL-EP, F.Cu at (250.4, 100.8)
- D1, L1, U3, USB1, USB2: moved to B.Cu
- U1: footprint RF_Module:ESP32-S3-WROOM-1 -> easyeda2kicad:ESP32-S3-WROOM-1; moved to B.Cu
- U4: value BQ25890RTWR -> BQ25890_1
- moved U3 140.1 mm to (186.3, 133.4)
- moved J1 138.6 mm to (205.7, 109.6), turned to 90 degrees
- moved U4 134.4 mm to (211.2, 100.8), turned to 90 degrees
- moved U1 130.7 mm to (179.4, 110.9), turned to 90 degrees
- moved C6 129.8 mm to (188.0, 128.2)
- moved D1 128.7 mm to (190.8, 133.1), turned to -90 degrees
- moved USB1 128.5 mm to (161.9, 122.0), turned to 90 degrees
- moved C8 123.2 mm to (184.2, 125.3), turned to 180 degrees
- moved R3 123.2 mm to (187.4, 132.2), turned to 180 degrees
- moved L1 122.4 mm to (188.5, 125.1), turned to 180 degrees
- moved C3 121.1 mm to (188.8, 126.4), turned to 180 degrees
- moved U2 120.5 mm to (161.9, 122.1), turned to 180 degrees
- moved C2 119.1 mm to (161.1, 132.6)
- moved C4 116.9 mm to (188.8, 124.2), turned to 180 degrees
- moved C10 115.4 mm to (182.9, 118.1), turned to 180 degrees
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Connections:
- J1 pad 1: unconnected-(J1-Pin_1-Pad1) -> GND
- J1 pad 2: unconnected-(J1-Pin_2-Pad2) -> Net-(J1-Pin_2)
- U1 pad 10: unconnected-(U1-IO17-Pad10) -> BUZZER
- U1 pad 11: unconnected-(U1-IO18-Pad11) -> SW_RIGHT
- U1 pad 12: unconnected-(U1-IO8-Pad12) -> SW_LEFT
- U1 pad 18: unconnected-(U1-IO10-Pad18) -> CE_6
- U1 pad 19: unconnected-(U1-IO11-Pad19) -> CE_5
- U1 pad 20: unconnected-(U1-IO12-Pad20) -> CE_4
- U1 pad 21: unconnected-(U1-IO13-Pad21) -> DISCHARGE_4
- U1 pad 22: unconnected-(U1-IO14-Pad22) -> DISCHARGE_5
- U1 pad 23: unconnected-(U1-IO21-Pad23) -> DISCHARGE_6
- U1 pad 24: unconnected-(U1-IO47-Pad24) -> MAIN_SDA
- U1 pad 25: unconnected-(U1-IO48-Pad25) -> MAIN_SCL
- U1 pad 28: unconnected-(U1-IO35-Pad28) -> TFT_SCL
- U1 pad 29: unconnected-(U1-IO36-Pad29) -> TFT_SDA
- U1 pad 30: unconnected-(U1-IO37-Pad30) -> TFT_RES
- U1 pad 31: unconnected-(U1-IO38-Pad31) -> TFT_DC
- U1 pad 32: unconnected-(U1-IO39-Pad32) -> TFT_BLK
- U1 pad 33: unconnected-(U1-IO40-Pad33) -> FAN
- U1 pad 34: unconnected-(U1-IO41-Pad34) -> DISCHARGE_1
- U1 pad 35: unconnected-(U1-IO42-Pad35) -> DISCHARGE_2
- U1 pad 36: unconnected-(U1-RXD0-Pad36) -> DISCHARGE_3
- U1 pad 37: unconnected-(U1-TXD0-Pad37) -> CE_1
- U1 pad 38: unconnected-(U1-IO2-Pad38) -> CE_2
- U1 pad 39: unconnected-(U1-IO1-Pad39) -> CE_3
- U4 pad 1: unconnected-(U4-VBUS-Pad1) -> VBUS
- U4 pad 10: unconnected-(U4-ILIM-Pad10) -> Net-(U4-ILIM)
- U4 pad 11: unconnected-(U4-TS-Pad11) -> Net-(U4-TS)
- U4 pad 13: unconnected-(U4-BAT-Pad13) -> Net-(Q2-S-Pad1)
- U4 pad 14: unconnected-(U4-BAT-Pad14) -> Net-(Q2-S-Pad1)
- U4 pad 15: unconnected-(U4-SYS-Pad15) -> SYS_1
- U4 pad 16: unconnected-(U4-SYS-Pad16) -> SYS_1
- U4 pad 17: unconnected-(U4-PGND-Pad17) -> GND
- U4 pad 18: unconnected-(U4-PGND-Pad18) -> GND
- U4 pad 19: unconnected-(U4-SW-Pad19) -> Net-(C13-Pad1)
- U4 pad 20: unconnected-(U4-SW-Pad20) -> Net-(C13-Pad1)
- U4 pad 21: unconnected-(U4-BTST-Pad21) -> Net-(U4-BTST)
- U4 pad 22: unconnected-(U4-REGN-Pad22) -> REGN_1
- U4 pad 23: unconnected-(U4-PMID-Pad23) -> Net-(U4-PMID)
- U4 pad 25: unconnected-(U4-PAD-Pad25) -> GND
- U4 pad 5: unconnected-(U4-SCL-Pad5) -> SCL_1
- U4 pad 6: unconnected-(U4-SDA-Pad6) -> SDA_1
- U4 pad 8: unconnected-(U4-OTG-Pad8) -> GND
- U4 pad 9: unconnected-(U4-~{CE}-Pad9) -> CE_1
Routing:
- net VBUS: track 0.00 -> 390.3 mm, vias 0 -> 33
- net +3.3V: track 0.00 -> 314.0 mm, vias 0 -> 9
- net GND: track 0.00 -> 114.0 mm, vias 0 -> 252
- net +5V: track 0.00 -> 106.4 mm, vias 0 -> 8
- net CE_6: track 0.00 -> 104.7 mm, vias 0 -> 1
- net DISCHARGE_3: track 0.00 -> 86.6 mm, vias 0 -> 2
- net CE_5: track 0.00 -> 85.5 mm, vias 0 -> 1
- net SDA_3: track 0.00 -> 78.9 mm, vias 0 -> 2
- net CE_3: track 0.00 -> 75.0 mm, vias 0 -> 1
- net SCL_3: track 0.00 -> 74.8 mm, vias 0 -> 2
- net DISCHARGE_6: track 0.00 -> 72.2 mm, vias 0 -> 1
- net DISCHARGE_2: track 0.00 -> 67.5 mm, vias 0 -> 2
- net CE_4: track 0.00 -> 66.1 mm, vias 0 -> 1
- net SDA_2: track 0.00 -> 58.9 mm, vias 0 -> 2
- net SDA_6: track 0.00 -> 58.6 mm, vias 0 -> 2
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- added copper zone on B.Cu, net +3.3V
- added copper zone on B.Cu, net GND
- added copper zone on F.Cu, net GND
Other:
- board outline added: 100 x 52 mm
- board text added: "1"
- board text added: "2"
- board text added: "3"
- board text added: ":3"
- board text added: "BOOT"
- board text added: "PRO"
- board text added: "WhoopDock 6"

Commit message: fixed PCB
Parts:
- added ?: , , F.Cu at (256.1, 128.6)
- added REF**: 1.3" TFT, easyeda2kicad:PowerPad, F.Cu at (256.2, 124.6)
Routing:
- net GND: track 114.0 -> 134.2 mm, vias 252 -> 270
- net MAIN_SCL: track 31.5 -> 33.4 mm, vias 1 -> 2
- net MAIN_SDA: track 29.1 -> 30.5 mm, vias 1 -> 2
- net +3.3V: track 314.0 -> 315.3 mm
- net VBUS: track 390.3 -> 389.8 mm, vias 33 -> 37
Other:
- board text added: "+"
- board text added: "-"
- board text added: "14v MAX"

Commit message: almost finalized except for readme
Parts:
- removed ?: , 
- removed REF**: 1.3" TFT, easyeda2kicad:PowerPad
