File: PCB/WhoopDock.kicad_sch (KiCad schematic)
At the start: 45 parts, among them J1 BetaFPV_BT2.0, J2 BetaFPV_BT2.0, J3 BetaFPV_BT2.0, J4 BetaFPV_BT2.0, J5 BetaFPV_BT2.0, J6 BetaFPV_BT2.0, SW1 SW_Push, U1 ESP32-S3-WROOM-1, U10 BQ25890RTWR, U2 CH224K, U3 XL1509-5.0E1, U4 BQ25890RTWR, U5 RT9193-33GB, U6 BQ25890RTWR, U7 BQ25890RTWR, U8 BQ25890RTWR, U9 BQ25890RTWR

Commit message: checkpoint
Parts:
- removed J2, J3, J4, J5, J6: BetaFPV_BT2.0, easyeda2kicad:BetaFPV BT2.0, symbol WhoopDock:BetaFPV_BT2.0
- removed U10, U6, U7, U8, U9: BQ25890RTWR, easyeda2kicad:WQFN-24_L4.0-W4.0-P0.50-BL-EP, symbol WhoopDock:BQ25890RTWR
- added C12, C14, C15, C16: 10uF, Capacitor_SMD:C_0805_2012Metric, symbol Device:C_Small
- added C13: 47nF, Capacitor_SMD:C_0603_1608Metric, symbol Device:C_Small
- added C17: 4.7uF, Capacitor_SMD:C_0603_1608Metric, symbol Device:C_Small
- added C18: 1uF, Capacitor_SMD:C_0603_1608Metric, symbol Device:C_Small
- added L2: 1.5uH, Inductor_SMD:L_APV_APH0420, symbol Device:L_Small
- added Q1: AO3400A, Package_TO_SOT_SMD:SOT-23, symbol Transistor_FET:AO3400A
- added Q2: AO4407A, easyeda2kicad:SOIC-8_L4.9-W3.9-P1.27-LS6.0-BL, symbol WhoopDock:AO4407A
- added R14, R25: 100, Resistor_SMD:R_0603_1608Metric, symbol Device:R_Small
- added R15, R16, R17, R24: 5.1k, Resistor_SMD:R_0603_1608Metric, symbol Device:R_Small
- added R18, R19: 10k, Resistor_SMD:R_0603_1608Metric, symbol Device:R_Small
- added R20, R21, R22, R23: 15, Resistor_SMD:R_2512_6332Metric, symbol Device:R_Small
- U4: value BQ25890RTWR -> BQ25890_1
Connections:
- net +3.3V: now also R15.2, R16.2, R17.2
- net GND: now also J1.1 (Pin_1), U4.17 (PGND), U4.18 (PGND), U4.25 (PAD), U4.8 (OTG), C12.1, C14.1, C15.1, C16.1, C17.1, C18.2, Q1.2 (S), Q2.4 (G), R14.1, R19.2, R24.1
- net VBUS: now also U4.1 (VBUS), C18.1
- net at J1.2 (Pin_2): now also C12.2, Q2.5 (D), Q2.6 (D), Q2.7 (D), Q2.8 (D), R20.2, R21.2, R22.2, R23.2
- net at U4.10 (ILIM): now also R14.2
- net at U4.11 (TS): now also R18.1, R19.1
- net at U4.13 (BAT): now also U4.14 (BAT), Q2.1 (S), Q2.2 (S), Q2.3 (S)
- net SYS_1: now reaches U4.15 (SYS)
- net SYS_1: now also U4.16 (SYS), C14.2, C15.2, L2.2
- net at U4.19 (SW): now also U4.20 (SW), C13.1, L2.1
- net at U4.21 (BTST): now also C13.2
- net REGN_1: now reaches U4.22 (REGN)
- net REGN_1: now also C17.2, R18.2
- net at U4.23 (PMID): now also C16.2
- net SCL_1: now reaches U4.5 (SCL)
- net SCL_1: now also R17.1
- net SDA_1: now reaches U4.6 (SDA)
- net SDA_1: now also R16.1
- net CE_1: now reaches U4.9 (~{CE})
- net CE_1: now also R15.1
- new net: Q1.1 (G), R24.2, R25.2
- new net: Q1.3 (D), R20.1, R21.1, R22.1, R23.1
- new net DISCHARGE_1: R25.1
- no-connect marks 5 -> 11
Other:
- moved on the sheet: J1, U4

Commit message: PCB Done
Parts:
- removed SW1: SW_Push, Button_Switch_THT:SW_PUSH_6mm_H5mm, symbol Switch:SW_Push
- added BUZZER1: MLT-8530, easyeda2kicad:BUZ-SMD_4P-L8.5-W8.5-P8.50-BR, symbol WhoopDock:MLT-8530
- added C19, C23, C24, C25, C26, C30, C31, C32, C33, C37, C38, C39, C40, C44, C45, C46, C47, C51, C52, C53, C54, C56, C58: 10uF, Capacitor_SMD:C_0805_2012Metric, symbol Device:C_Small
- added C20, C27, C34, C41, C48: 1uF, Capacitor_SMD:C_0603_1608Metric, symbol Device:C_Small
- added C21, C28, C35, C42, C49: 47nF, Capacitor_SMD:C_0603_1608Metric, symbol Device:C_Small
- added C22, C29, C36, C43, C50: 4.7uF, Capacitor_SMD:C_0603_1608Metric, symbol Device:C_Small
- added C55: 0.1uF, Capacitor_SMD:C_0603_1608Metric, symbol Device:C_Small
- added C57: 10nF, Capacitor_SMD:C_0603_1608Metric, symbol Device:C_Small
- added D2: 1N4148W, Diode_SMD:D_SOD-123F, symbol Diode:1N4148W
- added J2, J3, J4, J5, J6: BetaFPV_BT2.0, easyeda2kicad:BetaFPV BT2.0, symbol WhoopDock:BetaFPV_BT2.0
- added L3, L4, L5, L6, L7: 1.5uH, Inductor_SMD:L_APV_APH0420, symbol Device:L_Small
- added M1: Fan, easyeda2kicad:Fan, symbol Motor:Fan
- added Q10, Q12, Q14, Q6, Q8: AO4407A, easyeda2kicad:SOIC-8_L4.9-W3.9-P1.27-LS6.0-BL, symbol WhoopDock:AO4407A
- added Q11, Q13, Q3, Q4, Q5, Q7, Q9: AO3400A, Package_TO_SOT_SMD:SOT-23, symbol Transistor_FET:AO3400A
- added R26, R27, R28, R29, R40, R41, R52, R53, R64, R65, R76, R77: 100, Resistor_SMD:R_0603_1608Metric, symbol Device:R_Small
- added R30, R32, R38, R39, R42, R44, R50, R51, R54, R56, R62, R63, R66, R68, R74, R75, R78, R80, R86, R87, R88, R89, R90: 5.1k, Resistor_SMD:R_0603_1608Metric, symbol Device:R_Small
- added R31, R33, R43, R45, R55, R57, R67, R69, R79, R81: 10k, Resistor_SMD:R_0603_1608Metric, symbol Device:R_Small
- added R34, R35, R36, R37, R46, R47, R48, R49, R58, R59, R60, R61, R70, R71, R72, R73, R82, R83, R84, R85: 15, Resistor_SMD:R_2512_6332Metric, symbol Device:R_Small
- added R91: 0, Resistor_SMD:R_0603_1608Metric, symbol Device:R_Small
- added SW2, SW3: SW_Push, Button_Switch_THT:SW_PUSH_6mm_H5mm, symbol Switch:SW_Push
- added U10, U11, U12, U8, U9: BQ25890_1, easyeda2kicad:WQFN-24_L4.0-W4.0-P0.50-BL-EP, symbol WhoopDock:BQ25890RTWR
- added U13: RT9193-33GB, easyeda2kicad:SOT-23-5_L3.0-W1.7-P0.95-LS2.8-BL, symbol WhoopDock:RT9193-33GB
- added U6: ~, easyeda2kicad:1.3 TFT, symbol WhoopDock:TFT_1.3
- added U7: TCA9548APWR, Package_SO:TSSOP-24_4.4x7.8mm_P0.65mm, symbol Interface_Expansion:TCA9548APWR
- U1: footprint RF_Module:ESP32-S3-WROOM-1 -> easyeda2kicad:ESP32-S3-WROOM-1
Connections:
- net +3.3V: now also C54.2, C55.2, R32.2, R38.2, R39.2, R44.2, R50.2, R51.2, R56.2, R62.2, R63.2, R68.2, R74.2, R75.2, R80.2, R86.2, R87.2, R88.2, R89.2, R90.2, U7.24 (VCC)
- net +5V: now also BUZZER1.1 (+), C56.2, D2.1 (K), M1.1 (+), U13.1 (VIN), U13.3 (EN)
- net BOOT: now also R91.1
- net CE_1: now also U1.37 (TXD0)
- net DISCHARGE_1: now also U1.34 (IO41)
- net GND: now also C19.1, C20.2, C22.1, C23.1, C24.1, C25.1, C26.1, C27.2, C29.1, C30.1, C31.1, C32.1, C33.1, C34.2, C36.1, C37.1, C38.1, C39.1, C40.1, C41.2, C43.1, C44.1, C45.1, C46.1, C47.1, C48.2, C50.1, C51.1, C52.1, C53.1, C54.1, C55.1, C56.1, C57.1, C58.1, J2.1 (Pin_1), J3.1 (Pin_1), J4.1 (Pin_1), J5.1 (Pin_1), J6.1 (Pin_1), Q10.4 (G), Q11.2 (S), Q12.4 (G), Q13.2 (S), Q14.4 (G), Q3.2 (S), Q4.2 (S), Q5.2 (S), Q6.4 (G), Q7.2 (S), Q8.4 (G), Q9.2 (S), R29.1, R30.1, R31.2, R41.1, R42.1, R43.2, R53.1, R54.1, R55.2, R65.1, R66.1, R67.2, R77.1, R78.1, R79.2, R91.2, SW2.2, SW3.2, U10.17 (PGND), U10.18 (PGND), U10.25 (PAD), U10.8 (OTG), U11.17 (PGND), U11.18 (PGND), U11.25 (PAD), U11.8 (OTG), U12.17 (PGND), U12.18 (PGND), U12.25 (PAD), U12.8 (OTG), U13.2 (GND), U6.1 (GND), U7.1 (A0), U7.12 (GND), U7.2 (A1), U7.21 (A2), U8.17 (PGND), U8.18 (PGND), U8.25 (PAD), U8.8 (OTG), U9.17 (PGND), U9.18 (PGND), U9.25 (PAD), U9.8 (OTG)
- net SCL_1: now also U7.18 (SC6)
- net SDA_1: now also U7.17 (SD6)
- net VBUS: now also C20.1, C27.1, C34.1, C41.1, C48.1, U10.1 (VBUS), U11.1 (VBUS), U12.1 (VBUS), U8.1 (VBUS), U9.1 (VBUS)
- net at C12.2, J1.2 (Pin_2), Q2.5 (D)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: no longer R20.2, R21.2, R22.2, R23.2
- net at Q2.1 (S), Q2.2 (S), Q2.3 (S)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: now also R20.2, R21.2, R22.2, R23.2
- net BUZZER: now reaches U1.10 (IO17)
- net BUZZER: now also R26.1
- net SW_RIGHT: now reaches U1.11 (IO18)
- net SW_RIGHT: now also SW3.1
- net SW_LEFT: now reaches U1.12 (IO8)
- net SW_LEFT: now also SW2.1
- net CE_6: now reaches U1.18 (IO10)
- net CE_6: now also R80.1, U12.9 (~{CE})
- net CE_5: now reaches U1.19 (IO11)
- net CE_5: now also R68.1, U11.9 (~{CE})
- net CE_4: now reaches U1.20 (IO12)
- net CE_4: now also R56.1, U10.9 (~{CE})
- net DISCHARGE_4: now reaches U1.21 (IO13)
- net DISCHARGE_4: now also R52.1
- net DISCHARGE_5: now reaches U1.22 (IO14)
- net DISCHARGE_5: now also R64.1
- net DISCHARGE_6: now reaches U1.23 (IO21)
- net DISCHARGE_6: now also R76.1
- net MAIN_SDA: now reaches U1.24 (IO47)
- net MAIN_SDA: now also R89.1, U7.23 (SDA)
- net MAIN_SCL: now reaches U1.25 (IO48)
- net MAIN_SCL: now also R88.1, U7.22 (SCL)
- net TFT_SCL: now reaches U1.28 (IO35)
- net TFT_SCL: now also U6.3 (SCL)
- net TFT_SDA: now reaches U1.29 (IO36)
- net TFT_SDA: now also U6.4 (SDA)
- net TFT_RES: now reaches U1.30 (IO37)
- net TFT_RES: now also U6.5 (RES)
- net TFT_DC: now reaches U1.31 (IO38)
- net TFT_DC: now also U6.6 (DC)
- net TFT_BLK: now reaches U1.32 (IO39)
- net TFT_BLK: now also U6.7 (BLK)
- net FAN: now reaches U1.33 (IO40)
- net FAN: now also R27.1
- net DISCHARGE_2: now reaches U1.35 (IO42)
- net DISCHARGE_2: now also R28.1
- net DISCHARGE_3: now reaches U1.36 (RXD0)
- net DISCHARGE_3: now also R40.1
- net CE_2: now reaches U1.38 (IO2)
- net CE_2: now also R32.1, U8.9 (~{CE})
- net CE_3: now reaches U1.39 (IO1)
- net CE_3: now also R44.1, U9.9 (~{CE})
- new net: R29.2, U8.10 (ILIM)
- new net: R31.1, R33.1, U8.11 (TS)
- new net: Q6.1 (S), Q6.2 (S), Q6.3 (S), R34.2, R35.2, R36.2, R37.2, U8.13 (BAT), U8.14 (BAT)
- new net: C21.1, L3.1, U8.19 (SW), U8.20 (SW)
- new net: C21.2, U8.21 (BTST)
- new net: C23.2, U8.23 (PMID)
- new net: Q14.1 (S), Q14.2 (S), Q14.3 (S), R82.2, R83.2, R84.2, R85.2, U12.13 (BAT), U12.14 (BAT)
- new net: C47.2, J6.2 (Pin_2), Q14.5 (D), Q14.6 (D), Q14.7 (D), Q14.8 (D)
- new net: Q9.3 (D), R58.1, R59.1, R60.1, R61.1
- new net: Q10.1 (S), Q10.2 (S), Q10.3 (S), R58.2, R59.2, R60.2, R61.2, U10.13 (BAT), U10.14 (BAT)
- new net: Q11.3 (D), R70.1, R71.1, R72.1, R73.1
- new net: Q12.1 (S), Q12.2 (S), Q12.3 (S), R70.2, R71.2, R72.2, R73.2, U11.13 (BAT), U11.14 (BAT)
- new net: Q11.1 (G), R64.2, R66.2
- new net: R79.1, R81.1, U12.11 (TS)
- new net: Q7.3 (D), R46.1, R47.1, R48.1, R49.1
- new net: Q8.1 (S), Q8.2 (S), Q8.3 (S), R46.2, R47.2, R48.2, R49.2, U9.13 (BAT), U9.14 (BAT)
- new net: C19.2, J2.2 (Pin_2), Q6.5 (D), Q6.6 (D), Q6.7 (D), Q6.8 (D)
- new net: C30.2, U9.23 (PMID)
- new net: R55.1, R57.1, U10.11 (TS)
- new net: Q5.3 (D), R34.1, R35.1, R36.1, R37.1
- new net: C40.2, J5.2 (Pin_2), Q12.5 (D), Q12.6 (D), Q12.7 (D), Q12.8 (D)
- new net: R67.1, R69.1, U11.11 (TS)
- new net: R90.1, U7.3 (~{RESET})
- new net: M1.2 (-), Q4.3 (D)
- new net: C42.1, L6.1, U11.19 (SW), U11.20 (SW)
- new net: C42.2, U11.21 (BTST)
- new net: Q3.1 (G), R26.2
- new net: C26.2, J3.2 (Pin_2), Q8.5 (D), Q8.6 (D), Q8.7 (D), Q8.8 (D)
- new net: Q13.3 (D), R82.1, R83.1, R84.1, R85.1
- new net: Q13.1 (G), R76.2, R78.2
- new net: R41.2, U9.10 (ILIM)
- new net: C57.2, U13.4 (BP)
- new net: BUZZER1.2, BUZZER1.3, BUZZER1.4, D2.2 (A), Q3.3 (D)
- new net: Q7.1 (G), R40.2, R42.2
- new net: R43.1, R45.1, U9.11 (TS)
- new net: R53.2, U10.10 (ILIM)
- new net: C33.2, J4.2 (Pin_2), Q10.5 (D), Q10.6 (D), Q10.7 (D), Q10.8 (D)
- new net: C51.2, U12.23 (PMID)
- new net: R65.2, U11.10 (ILIM)
- new net: C35.1, L5.1, U10.19 (SW), U10.20 (SW)
- new net: C35.2, U10.21 (BTST)
- new net: C28.1, L4.1, U9.19 (SW), U9.20 (SW)
- new net: C28.2, U9.21 (BTST)
- new net: Q9.1 (G), R52.2, R54.2
- new net: Q5.1 (G), R28.2, R30.2
- new net: Q4.1 (G), R27.2
- new net: C44.2, U11.23 (PMID)
- new net: C49.1, L7.1, U12.19 (SW), U12.20 (SW)
- new net: C49.2, U12.21 (BTST)
- new net: R77.2, U12.10 (ILIM)
- new net: C37.2, U10.23 (PMID)
- new net +3.3V(LCD): C58.2, U13.5 (VOUT), U6.2 (VCC)
- new net REGN_2: C22.2, R33.2, U8.22 (REGN)
- new net REGN_3: C29.2, R45.2, U9.22 (REGN)
- new net REGN_4: C36.2, R57.2, U10.22 (REGN)
- new net REGN_5: C43.2, R69.2, U11.22 (REGN)
- new net REGN_6: C50.2, R81.2, U12.22 (REGN)
- new net SCL_2: R39.1, U7.16 (SC5), U8.5 (SCL)
- new net SCL_3: R51.1, U7.14 (SC4), U9.5 (SCL)
- new net SCL_4: R63.1, U10.5 (SCL), U7.7 (SC1)
- new net SCL_5: R75.1, U11.5 (SCL), U7.9 (SC2)
- new net SCL_6: R87.1, U12.5 (SCL), U7.11 (SC3)
- new net SDA_2: R38.1, U7.15 (SD5), U8.6 (SDA)
- new net SDA_3: R50.1, U7.13 (SD4), U9.6 (SDA)
- new net SDA_4: R62.1, U10.6 (SDA), U7.6 (SD1)
- new net SDA_5: R74.1, U11.6 (SDA), U7.8 (SD2)
- new net SDA_6: R86.1, U12.6 (SDA), U7.10 (SD3)
- new net SYS_2: C24.2, C25.2, L3.2, U8.15 (SYS), U8.16 (SYS)
- new net SYS_3: C31.2, C32.2, L4.2, U9.15 (SYS), U9.16 (SYS)
- new net SYS_4: C38.2, C39.2, L5.2, U10.15 (SYS), U10.16 (SYS)
- new net SYS_5: C45.2, C46.2, L6.2, U11.15 (SYS), U11.16 (SYS)
- new net SYS_6: C52.2, C53.2, L7.2, U12.15 (SYS), U12.16 (SYS)
- no-connect marks 11 -> 48
Other:
- note added: "3.3V LDO 1"
- note added: "3.3V LDO 2"
- note added: "Channel 1"
- note added: "Channel 2"
- note added: "Channel 3"
- note added: "Channel 4"
- note added: "Channel 5"
- note added: "Channel 6"
- note removed: "3.3V LDO"
- moved on the sheet: C12, C13, C14, C15, C16, C17, C18, J1, L2, Q1, Q2, R14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

Commit message: almost finalized except for readme
Parts:
- C1, C12, C14, C15, C16, C19, C23, C24, C25, C26, C30, C31, C32, C33, C37, C38, C39, C40, C44, C45, C46, C47, C5, C51, C52, C53, C54, C56, C58, C7, C9: LCSC Part (none) -> C440198
- C10, C11, C18, C20, C27, C34, C41, C48: LCSC Part (none) -> C15849
- C13, C21, C28, C35, C42, C49: LCSC Part (none) -> C1622
- C17, C22, C29, C36, C43, C50: LCSC Part (none) -> C19666
- C2, C55, C6: LCSC Part (none) -> C14663
- C3, C4: LCSC Part (none) -> C561794
- C57, C8: LCSC Part (none) -> C57112
- D1: LCSC Part (none) -> C2480
- D2: LCSC Part (none) -> C108804
- L1: LCSC Part (none) -> C2894721
- L2, L3, L4, L5, L6, L7: LCSC Part (none) -> C167205
- Q1, Q11, Q13, Q3, Q4, Q5, Q7, Q9: LCSC Part (none) -> C20917
- R1, R15, R16, R17, R2, R24, R30, R32, R38, R39, R42, R44, R50, R51, R54, R56, R62, R63, R66, R68, R74, R75, R78, R80, R86, R87, R88, R89, R90: LCSC Part (none) -> C23186
- R10: LCSC Part (none) -> C21190
- R11, R12, R13, R18, R19, R3, R31, R33, R4, R43, R45, R5, R55, R57, R67, R69, R79, R81, R9: LCSC Part (none) -> C25804
- R14, R25, R26, R27, R28, R29, R40, R41, R52, R53, R64, R65, R76, R77: LCSC Part (none) -> C22775
- R20, R21, R22, R23, R34, R35, R36, R37, R46, R47, R48, R49, R58, R59, R60, R61, R70, R71, R72, R73, R82, R83, R84, R85: LCSC Part (none) -> C20087
- SW2, SW3: LCSC Part (none) -> C2837531
- U1: LCSC Part (none) -> C2913198
- U2: LCSC Part (none) -> C970725
- U7: LCSC Part (none) -> C130026
Other:
- note added: "Buzzer, Fan, Buttons and Display"
- note added: "I2C Multiplexer"
- note added: "MCU"
- title: (none) -> WhoopDock 6 Pro
- moved on the sheet: BUZZER1, C10, C12, C13, C14, C15, C16, C17, C18, C19, C20, C21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
